File: LLC CONVERTER/_autosave-LLC CONVERTER.kicad_pcb (KiCad board)
At the start: 2 copper layers, 23 parts, among them IC1 UCC256601DDBR

Commit message: first commit
Parts:
- added C4: C, Capacitor_THT:C_Rect_L13.5mm_W5.0mm_P10.00mm_FKS3_FKP3_MKS4, F.Cu at (126.8, 62.8)
- added FL1: PH9455x105NL, Inductor_THT:L_CommonMode_PulseElectronics_PH9455x105NL_1, F.Cu at (107.7, 63.9)
- added TH2: NTC, Resistor_THT:R_Bare_Metal_Element_L12.4mm_W4.8mm_P11.40mm, F.Cu at (126.5, 56.3)
Connections:
- D1 pad 2: Net-(D1-A) -> unconnected-(D1-A-Pad2)
- D2 pad 2: Net-(D2-A) -> unconnected-(D2-A-Pad2)
- LINE1 pad 1: Net-(D1-A) -> Net-(LINE1-Pin_1)
- LINE1 pad 2: (no net) -> Net-(LINE1-Pin_1)
- NEUTRAL1 pad 1: Net-(D2-A) -> Net-(NEUTRAL1-Pin_1)
- NEUTRAL1 pad 2: (no net) -> Net-(NEUTRAL1-Pin_1)
